File: qaz/qaz.kicad_pcb (KiCad board)
At the start: 2 copper layers, 217.3 x 57.1 mm, 47 parts, among them J1 OLED-128x32, SW1 SW_Push, SW10 SW_Push, SW11 SW_Push, SW12 SW_Push, SW13 SW_Push, SW14 SW_Push, SW15 SW_Push, SW16 SW_Push, SW17 SW_Push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

Commit message: .
Parts:
- added REF**: MountingHole_2.2mm_M2_ISO7380_Pad, MountingHole:MountingHole_2.2mm_M2_ISO7380_Pad, F.Cu at (271.2, 72.5)
- added REF**: MountingHole_2.2mm_M2_ISO7380_Pad, MountingHole:MountingHole_2.2mm_M2_ISO7380_Pad, F.Cu at (271.2, 40.8)
- SW1, SW10, SW12, SW13, SW14, SW15, SW16, SW17, SW18, SW2, SW21, SW22, SW23, SW25, SW26, SW27, SW28, SW3, SW4, SW5, SW6, SW7, SW8, SW9: footprint Button_Switch_Keyboard:SW_Cherry_MX_1.00u_PCB -> MCU:SW_Cherry_MX_1.00u_PCB_fixed
- SW11: footprint Button_Switch_Keyboard:SW_Cherry_MX_1.25u_PCB -> MCU:SW_Cherry_MX_1.00u_PCB_fixed
- SW19: footprint Button_Switch_Keyboard:SW_Cherry_MX_1.75u_PCB -> MCU:SW_Cherry_MX_1.00u_PCB_fixed
- SW20, SW24: footprint Button_Switch_Keyboard:SW_Cherry_MX_1.50u_PCB -> MCU:SW_Cherry_MX_1.00u_PCB_fixed
- moved J1 0.42 mm to (251.9, 68.9)
Routing:
- net r2: track 191.3 -> 248.8 mm
- net r0: track 156.9 -> 189.1 mm, vias 0 -> 2
- net Net-(D6-A-Pad1): track 0.00 -> 9.93 mm
- net c0: track 245.8 -> 245.3 mm
Other:
- board size 217.3 x 57.1 mm -> 223.6 x 57.1 mm
- board text added: "MICRO QAZ"

Commit message: .
Routing:
- net r2: track 248.8 -> 251.3 mm
- net r0: track 189.1 -> 187.7 mm
- net c1: track 213.6 -> 212.3 mm
- net c3: track 173.4 -> 172.1 mm
- net c7: track 96.5 -> 95.1 mm
- net r1: track 181.3 -> 180.0 mm
- net c2: track 193.5 -> 192.5 mm
- net c6: track 114.8 -> 113.9 mm
- net c4: track 155.3 -> 154.3 mm
- net c5: track 112.2 -> 111.4 mm
- net c0: track 245.3 -> 244.6 mm
- net c8: track 71.7 -> 71.0 mm
