File: qaz/qaz.kicad_pcb (KiCad board)
At the start: 2 copper layers, 223.6 x 57.1 mm, 49 parts, among them J1 OLED-128x32, SW1 SW_Push, SW10 SW_Push, SW11 SW_Push, SW12 SW_Push, SW13 SW_Push, SW14 SW_Push, SW15 SW_Push, SW16 SW_Push, SW17 SW_Push, SW18 SW_Push, SW19 SW_Push, SW2 SW_Push, SW20 SW_Push, SW21 SW_Push, SW22 SW_Push, SW23 SW_Push, SW24 SW_Push, SW25 SW_Push, SW26 SW_Push, SW27 SW_Push, SW28 SW_Push, SW3 SW_Push, SW4 SW_Push, SW5 SW_Push, SW6 SW_Push, SW7 SW_Push, SW8 SW_Push, SW9 SW_Push, U1 rp2040-zero

Commit message: .
Parts:
- removed J1: OLED-128x32, MCU:OLED-128x32
- removed the REF** at (271.2, 72.5)
- removed the REF** at (54.0, 72.6)
- removed the REF** at (271.2, 40.8)
- added REF**: MountingHole_2.2mm_M2_ISO7380_Pad, MountingHole:MountingHole_2.2mm_M2_ISO7380_Pad, F.Cu at (241.7, 35.7)
- added REF**: MountingHole_2.2mm_M2_ISO7380_Pad, MountingHole:MountingHole_2.2mm_M2_ISO7380_Pad, F.Cu at (21.4, 71.4)
- added REF**: MountingHole_2.2mm_M2_ISO7380_Pad, MountingHole:MountingHole_2.2mm_M2_ISO7380_Pad, F.Cu at (241.7, 71.4)
- D1, D10, D11, D12, D13, D14, D15, D2, D3, D4, D5, D6, D7, D8, D9: footprint Package_TO_SOT_SMD:SOT-23 -> custom:bav70
- SW1, SW10, SW11, SW12, SW13, SW14, SW15, SW16, SW17, SW18, SW19, SW2, SW20, SW21, SW22, SW23, SW24, SW25, SW26, SW27, SW28, SW3, SW4, SW5, SW6, SW7, SW8, SW9: footprint MCU:SW_Cherry_MX_1.00u_PCB_fixed -> PCM_marbastlib-xp-choc:SW_choc_MxCombo_1u
- U1: moved to F.Cu
- moved SW12 34.7 mm to (58.3, 53.6)
- moved SW15 34.7 mm to (115.5, 53.6)
- moved SW1 34.7 mm to (34.5, 34.5)
- moved SW11 34.7 mm to (36.9, 53.6)
- moved SW13 34.7 mm to (77.4, 53.6)
- moved SW14 34.7 mm to (96.4, 53.6)
- moved SW16 34.7 mm to (134.5, 53.6)
- moved SW17 34.7 mm to (153.6, 53.6)
- moved SW18 34.7 mm to (172.6, 53.6)
- moved SW19 34.7 mm to (198.8, 53.6)
- moved SW20 34.7 mm to (39.3, 72.6)
- moved SW21 34.7 mm to (63.1, 72.6)
- moved SW10 34.7 mm to (206.0, 34.5)
- moved SW2 34.7 mm to (53.6, 34.5)
- moved SW22 34.7 mm to (82.2, 72.6)
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Connections:
- D13 pad 2: unconnected-(D13-A-Pad2) -> Net-(D13-A-Pad2)
- D15 pad 2: Net-(D15-A-Pad2) -> unconnected-(D15-A-Pad2)
- SW25 pad 1: Net-(D14-A-Pad1) -> Net-(D13-A-Pad2)
- SW25 pad 2: c6 -> c5
- SW26 pad 1: Net-(D14-A-Pad2) -> Net-(D14-A-Pad1)
- SW26 pad 2: c7 -> c6
- SW27 pad 1: Net-(D15-A-Pad1) -> Net-(D14-A-Pad2)
- SW27 pad 2: c8 -> c7
- SW28 pad 1: Net-(D15-A-Pad2) -> Net-(D15-A-Pad1)
- SW28 pad 2: c9 -> c8
- U1 pad 1: c1 -> c8
- U1 pad 10: r0 -> r2
- U1 pad 11: r1 -> r0
- U1 pad 12: r2 -> r1
- U1 pad 13: sda -> unconnected-(U1-12-Pad13)
- U1 pad 14: scl -> unconnected-(U1-13-Pad14)
- U1 pad 2: c2 -> c7
- U1 pad 20: c0 -> c9
- U1 pad 21: +3.3V -> unconnected-(U1-3V3-Pad21)
- U1 pad 3: c3 -> c6
- U1 pad 4: c4 -> c5
- U1 pad 5: c5 -> c4
- U1 pad 6: c6 -> c3
- U1 pad 7: c7 -> c2
- U1 pad 8: c8 -> c1
- U1 pad 9: c9 -> c0
Routing:
- net c4: track 154.3 -> 549.1 mm, vias 0 -> 2
- net c5: track 111.4 -> 448.0 mm, vias 0 -> 2
- net c3: track 172.1 -> 484.4 mm, vias 0 -> 2
- net c6: track 113.9 -> 358.3 mm, vias 0 -> 2
- net c2: track 192.5 -> 425.6 mm, vias 0 -> 2
- net r0: track 187.7 -> 395.0 mm, vias 2 -> 1
- net c7: track 95.1 -> 267.8 mm, vias 0 -> 2
- net c1: track 212.3 -> 367.3 mm, vias 0 -> 2
- net r2: track 251.3 -> 395.8 mm, vias 0 -> 1
- net c8: track 71.0 -> 149.6 mm, vias 0 -> 2
- net c0: track 244.6 -> 299.9 mm
- net c9: track 53.9 -> 12.9 mm, vias 1 -> 0
- net sda: track 14.9 -> 0.00 mm
- net scl: track 14.9 -> 0.00 mm
- net Net-(D15-A-Pad2): track 12.5 -> 0.00 mm
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- added copper zone on B.Cu, net (none)
- added copper zone on F.Cu, net (none)
- removed copper zone on F.Cu, net +3.3V
- removed copper zone on B.Cu, net GND
Other:
- board size 223.6 x 57.1 mm -> 227.4 x 57.3 mm
- board text removed: "MICRO QAZ"

Commit message: .
Parts:
- added J1: OLED-128x32, custom:OLED-128x32, F.Cu at (221.3, 79.6)
Connections:
- U1 pad 13: unconnected-(U1-12-Pad13) -> scl
- U1 pad 14: unconnected-(U1-13-Pad14) -> sda
- U1 pad 21: unconnected-(U1-3V3-Pad21) -> +3.3V
Routing:
- net GND: track 0.00 -> 61.1 mm, vias 0 -> 2
- net +3.3V: track 0.00 -> 54.6 mm, vias 0 -> 2
- net sda: track 0.00 -> 31.6 mm
- net scl: track 0.00 -> 31.6 mm
- net c6: track 358.3 -> 357.3 mm
- net c7: track 267.8 -> 266.9 mm
- net c5: track 448.0 -> 447.0 mm
- net c4: track 549.1 -> 548.4 mm
- net c1: track 367.3 -> 366.7 mm
