File: qaz/qaz.kicad_sch (KiCad schematic)
At the start: 45 parts, among them J1 OLED-128x32, SW1 SW_Push, SW10 SW_Push, SW11 SW_Push, SW12 SW_Push, SW13 SW_Push, SW14 SW_Push, SW15 SW_Push, SW16 SW_Push, SW17 SW_Push, SW18 SW_Push, SW19 SW_Push, SW2 SW_Push, SW20 SW_Push, SW21 SW_Push, SW22 SW_Push, SW23 SW_Push, SW24 SW_Push, SW25 SW_Push, SW26 SW_Push, SW27 SW_Push, SW28 SW_Push, SW3 SW_Push, SW4 SW_Push, SW5 SW_Push, SW6 SW_Push, SW7 SW_Push, SW8 SW_Push, SW9 SW_Push, U1 rp2040-zero

Commit message: .
Parts:
- SW1, SW10, SW12, SW13, SW14, SW15, SW16, SW17, SW18, SW2, SW21, SW22, SW23, SW25, SW26, SW27, SW28, SW3, SW4, SW5, SW6, SW7, SW8, SW9: footprint Button_Switch_Keyboard:SW_Cherry_MX_1.00u_PCB -> MCU:SW_Cherry_MX_1.00u_PCB_fixed
- SW11: footprint Button_Switch_Keyboard:SW_Cherry_MX_1.25u_PCB -> MCU:SW_Cherry_MX_1.00u_PCB_fixed
- SW19: footprint Button_Switch_Keyboard:SW_Cherry_MX_1.75u_PCB -> MCU:SW_Cherry_MX_1.00u_PCB_fixed
- SW20, SW24: footprint Button_Switch_Keyboard:SW_Cherry_MX_1.50u_PCB -> MCU:SW_Cherry_MX_1.00u_PCB_fixed
Changed lines of the file:
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@@
       (effects (font (size 1.27 1.27)))
     )
-    (property "Footprint" "Button_Switch_Keyboard:SW_Cherry_MX_1.25u_PCB" (at 104.14 67.31 0)
+    (property "Footprint" "MCU:SW_Cherry_MX_1.00u_PCB_fixed" (at 104.14 67.31 0)
       (effects (font (size 1.27 1.27)) hide)
     )
@@
       (effects (font (size 1.27 1.27)))
     )
-    (property "Footprint" "Button_Switch_Keyboard:SW_Cherry_MX_1.00u_PCB" (at 195.58 39.37 0)
+    (property "Footprint" "MCU:SW_Cherry_MX_1.00u_PCB_fixed" (at 195.58 39.37 0)
       (effects (font (size 1.27 1.27)) hide)
     )
@@
       (effects (font (size 1.27 1.27)))
     )
-    (property "Footprint" "Button_Switch_Keyboard:SW_Cherry_MX_1.00u_PCB" (at 134.62 39.37 0)
+    (property "Footprint" "MCU:SW_Cherry_MX_1.00u_PCB_fixed" (at 134.62 39.37 0)
       (effects (font (size 1.27 1.27)) hide)
     )
@@
       (effects (font (size 1.27 1.27)))
     )
-    (property "Footprint" "Button_Switch_Keyboard:SW_Cherry_MX_1.00u_PCB" (at 119.38 67.31 0)
+    (property "Footprint" "MCU:SW_Cherry_MX_1.00u_PCB_fixed" (at 119.38 67.31 0)
       (effects (font (size 1.27 1.27)) hide)
     )
@@
       (effects (font (size 1.27 1.27)))
     )
-    (property "Footprint" "Button_Switch_Keyboard:SW_Cherry_MX_1.00u_PCB" (at 195.58 67.31 0)
+    (property "Footprint" "MCU:SW_Cherry_MX_1.00u_PCB_fixed" (at 195.58 67.31 0)
       (effects (font (size 1.27 1.27)) hide)
     )
@@
       (effects (font (size 1.27 1.27)))
     )
-    (property "Footprint" "Button_Switch_Keyboard:SW_Cherry_MX_1.00u_PCB" (at 226.06 39.37 0)
+    (property "Footprint" "MCU:SW_Cherry_MX_1.00u_PCB_fixed" (at 226.06 39.37 0)
       (effects (font (size 1.27 1.27)) hide)
     )
@@
       (effects (font (size 1.27 1.27)))
     )
-    (property "Footprint" "Button_Switch_Keyboard:SW_Cherry_MX_1.00u_PCB" (at 149.86 39.37 0)
+    (property "Footprint" "MCU:SW_Cherry_MX_1.00u_PCB_fixed" (at 149.86 39.37 0)
       (effects (font (size 1.27 1.27)) hide)
     )
@@
       (effects (font (size 1.27 1.27)))
     )
-    (property "Footprint" "Button_Switch_Keyboard:SW_Cherry_MX_1.00u_PCB" (at 134.62 67.31 0)
+    (property "Footprint" "MCU:SW_Cherry_MX_1.00u_PCB_fixed" (at 134.62 67.31 0)
       (effects (font (size 1.27 1.27)) hide)
     )
@@
       (effects (font (size 1.27 1.27)))
     )
-    (property "Footprint" "Button_Switch_Keyboard:SW_Cherry_MX_1.50u_PCB" (at 165.1 95.25 0)
+    (property "Footprint" "MCU:SW_Cherry_MX_1.00u_PCB_fixed" (at 165.1 95.25 0)
       (effects (font (size 1.27 1.27)) hide)
     )
@@
       (effects (font (size 1.27 1.27)))
     )
-    (property "Footprint" "Button_Switch_Keyboard:SW_Cherry_MX_1.00u_PCB" (at 210.82 67.31 0)
+    (property "Footprint" "MCU:SW_Cherry_MX_1.00u_PCB_fixed" (at 210.82 67.31 0)
       (effects (font (size 1.27 1.27)) hide)
     )
@@
       (effects (font (size 1.27 1.27)))
     )
-    (property "Footprint" "Button_Switch_Keyboard:SW_Cherry_MX_1.00u_PCB" (at 165.1 39.37 0)
+    (property "Footprint" "MCU:SW_Cherry_MX_1.00u_PCB_fixed" (at 165.1 39.37 0)
       (effects (font (size 1.27 1.27)) hide)
     )
@@
       (effects (font (size 1.27 1.27)))
     )
-    (property "Footprint" "Button_Switch_Keyboard:SW_Cherry_MX_1.00u_PCB" (at 165.1 67.31 0)
+    (property "Footprint" "MCU:SW_Cherry_MX_1.00u_PCB_fixed" (at 165.1 67.31 0)
       (effects (font (size 1.27 1.27)) hide)
     )
@@
       (effects (font (size 1.27 1.27)))
     )
-    (property "Footprint" "Button_Switch_Keyboard:SW_Cherry_MX_1.00u_PCB" (at 149.86 95.25 0)
+    (property "Footprint" "MCU:SW_Cherry_MX_1.00u_PCB_fixed" (at 149.86 95.25 0)
       (effects (font (size 1.27 1.27)) hide)
     )
@@
       (effects (font (size 1.27 1.27)))
     )
-    (property "Footprint" "Button_Switch_Keyboard:SW_Cherry_MX_1.75u_PCB" (at 226.06 67.31 0)
+    (property "Footprint" "MCU:SW_Cherry_MX_1.00u_PCB_fixed" (at 226.06 67.31 0)
       (effects (font (size 1.27 1.27)) hide)
     )
@@
       (effects (font (size 1.27 1.27)))
     )
-    (property "Footprint" "Button_Switch_Keyboard:SW_Cherry_MX_1.00u_PCB" (at 180.34 39.37 0)
+    (property "Footprint" "MCU:SW_Cherry_MX_1.00u_PCB_fixed" (at 180.34 39.37 0)
       (effects (font (size 1.27 1.27)) hide)
     )
@@
       (effects (font (size 1.27 1.27)))
     )
-    (property "Footprint" "Button_Switch_Keyboard:SW_Cherry_MX_1.00u_PCB" (at 226.06 95.25 0)
+    (property "Footprint" "MCU:SW_Cherry_MX_1.00u_PCB_fixed" (at 226.06 95.25 0)
       (effects (font (size 1.27 1.27)) hide)
     )
@@
       (effects (font (size 1.27 1.27)))
     )
-    (property "Footprint" "Button_Switch_Keyboard:SW_Cherry_MX_1.00u_PCB" (at 241.3 95.25 0)
+    (property "Footprint" "MCU:SW_Cherry_MX_1.00u_PCB_fixed" (at 241.3 95.25 0)
       (effects (font (size 1.27 1.27)) hide)
     )
@@
       (effects (font (size 1.27 1.27)))
     )
-    (property "Footprint" "Button_Switch_Keyboard:SW_Cherry_MX_1.00u_PCB" (at 210.82 39.37 0)
+    (property "Footprint" "MCU:SW_Cherry_MX_1.00u_PCB_fixed" (at 210.82 39.37 0)
       (effects (font (size 1.27 1.27)) hide)
     )
@@
       (effects (font (size 1.27 1.27)))
     )
-    (property "Footprint" "Button_Switch_Keyboard:SW_Cherry_MX_1.00u_PCB" (at 149.86 67.31 0)
+    (property "Footprint" "MCU:SW_Cherry_MX_1.00u_PCB_fixed" (at 149.86 67.31 0)
       (effects (font (size 1.27 1.27)) hide)
     )
@@
       (effects (font (size 1.27 1.27)))
     )
-    (property "Footprint" "Button_Switch_Keyboard:SW_Cherry_MX_1.00u_PCB" (at 134.62 95.25 0)
+    (property "Footprint" "MCU:SW_Cherry_MX_1.00u_PCB_fixed" (at 134.62 95.25 0)
       (effects (font (size 1.27 1.27)) hide)
     )
@@
       (effects (font (size 1.27 1.27)))
     )
-    (property "Footprint" "Button_Switch_Keyboard:SW_Cherry_MX_1.00u_PCB" (at 210.82 95.25 0)
+    (property "Footprint" "MCU:SW_Cherry_MX_1.00u_PCB_fixed" (at 210.82 95.25 0)
       (effects (font (size 1.27 1.27)) hide)
     )
@@
       (effects (font (size 1.27 1.27)))
     )
-    (property "Footprint" "Button_Switch_Keyboard:SW_Cherry_MX_1.00u_PCB" (at 241.3 39.37 0)
+    (property "Footprint" "MCU:SW_Cherry_MX_1.00u_PCB_fixed" (at 241.3 39.37 0)
       (effects (font (size 1.27 1.27)) hide)
     )
@@
       (effects (font (size 1.27 1.27)))
     )
-    (property "Footprint" "Button_Switch_Keyboard:SW_Cherry_MX_1.00u_PCB" (at 104.14 39.37 0)
+    (property "Footprint" "MCU:SW_Cherry_MX_1.00u_PCB_fixed" (at 104.14 39.37 0)
       (effects (font (size 1.27 1.27)) hide)
     )
@@
       (effects (font (size 1.27 1.27)))
     )
-    (property "Footprint" "Button_Switch_Keyboard:SW_Cherry_MX_1.00u_PCB" (at 195.58 95.25 0)
+    (property "Footprint" "MCU:SW_Cherry_MX_1.00u_PCB_fixed" (at 195.58 95.25 0)
       (effects (font (size 1.27 1.27)) hide)
     )
@@
       (effects (font (size 1.27 1.27)))
     )
-    (property "Footprint" "Button_Switch_Keyboard:SW_Cherry_MX_1.50u_PCB" (at 104.14 95.25 0)
+    (property "Footprint" "MCU:SW_Cherry_MX_1.00u_PCB_fixed" (at 104.14 95.25 0)
       (effects (font (size 1.27 1.27)) hide)
     )
@@
       (effects (font (size 1.27 1.27)))
     )
-    (property "Footprint" "Button_Switch_Keyboard:SW_Cherry_MX_1.00u_PCB" (at 180.34 67.31 0)
+    (property "Footprint" "MCU:SW_Cherry_MX_1.00u_PCB_fixed" (at 180.34 67.31 0)
       (effects (font (size 1.27 1.27)) hide)
     )
@@
       (effects (font (size 1.27 1.27)))
     )
-    (property "Footprint" "Button_Switch_Keyboard:SW_Cherry_MX_1.00u_PCB" (at 119.38 39.37 0)
+    (property "Footprint" "MCU:SW_Cherry_MX_1.00u_PCB_fixed" (at 119.38 39.37 0)
       (effects (font (size 1.27 1.27)) hide)
     )
@@
       (effects (font (size 1.27 1.27)))
     )
-    (property "Footprint" "Button_Switch_Keyboard:SW_Cherry_MX_1.00u_PCB" (at 119.38 95.25 0)
-      (effects (font (size 1.27 1.27)) hide)
-    )
+    (property "Footprint" "MCU:SW_Cherry_MX_1.00u_PCB_fixed" (at 119.38 95.25 0)
+      (effects (font (size 1.27 1.27)) hide)
+    )

Commit message: .
Parts:
- removed J1: OLED-128x32, MCU:OLED-128x32, symbol display:OLED-128x32
- D1, D10, D11, D12, D13, D14, D15, D2, D3, D4, D5, D6, D7, D8, D9: footprint Package_TO_SOT_SMD:SOT-23 -> custom:bav70
- SW1, SW10, SW11, SW12, SW13, SW14, SW15, SW16, SW17, SW18, SW19, SW2, SW20, SW21, SW22, SW23, SW24, SW25, SW26, SW27, SW28, SW3, SW4, SW5, SW6, SW7, SW8, SW9: footprint MCU:SW_Cherry_MX_1.00u_PCB_fixed -> PCM_marbastlib-xp-choc:SW_choc_MxCombo_1u
Connections:
- net c0: now also U1.9 (8); no longer U1.20 (29)
- net c1: now also U1.8 (7); no longer U1.1 (0)
- net c2: now also U1.7 (6); no longer U1.2 (1)
- net c3: now also U1.6 (5); no longer U1.3 (2)
- net c4: now also U1.5 (4); no longer U1.4 (3)
- net c5: now also SW25.2, U1.4 (3); no longer U1.5 (4)
- net c6: now also SW26.2, U1.3 (2); no longer SW25.2, U1.6 (5)
- net c7: now also SW27.2, U1.2 (1); no longer SW26.2, U1.7 (6)
- net c8: now also SW28.2, U1.1 (0); no longer SW27.2, U1.8 (7)
- net c9: now also U1.20 (29); no longer SW28.2, U1.9 (8)
- net r0: now also U1.11 (10); no longer U1.10 (9)
- net r1: now also U1.12 (11); no longer U1.11 (10)
- net r2: now also U1.10 (9); no longer U1.12 (11)
- net at D14.1 (A): now also SW26.1; no longer SW25.1
- net at D14.2 (A): now also SW27.1; no longer SW26.1
- net at D13.2 (A): now also SW25.1
- net at D15.1 (A): now also SW28.1; no longer SW27.1
- net at D15.2 (A): no longer SW28.1
- net +3.3V: no longer names the net of U1.21 (3V3)
- net scl: no longer names the net of U1.14 (13)
- net sda: no longer names the net of U1.13 (12)
Other:
- moved on the sheet: SW25, SW26, SW27, SW28

Commit message: .
Parts:
- added J1: OLED-128x32, custom:OLED-128x32, symbol display:OLED-128x32
Connections:
- net GND: now also J1.1 (GND)
- net scl: now reaches U1.13 (12)
- net scl: now also J1.3 (SCL)
- net sda: now reaches U1.14 (13)
- net sda: now also J1.4 (SDA)
- net +3.3V: now reaches U1.21 (3V3)
- net +3.3V: now also J1.2 (VCC)
Changed lines of the file:
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@@
+    )
+  )
+  (global_label "scl" (shape input) (at 53.34 99.06 180) (fields_autoplaced)
+    (effects (font (size 1.27 1.27)) (justify right))
+    (property "Intersheetrefs" "${INTERSHEET_REFS}" (at 47.5729 99.06 0)
+      (effects (font (size 1.27 1.27)) (justify right) hide)
     )
   )
@@
     (property "Intersheetrefs" "${INTERSHEET_REFS}" (at 76.4033 62.23 0)
       (effects (font (size 1.27 1.27)) (justify left) hide)
+    )
+  )
+  (global_label "sda" (shape input) (at 53.34 80.01 270) (fields_autoplaced)
+    (effects (font (size 1.27 1.27)) (justify right))
+    (property "Intersheetrefs" "${INTERSHEET_REFS}" (at 53.34 86.3213 90)
+      (effects (font (size 1.27 1.27)) (justify right) hide)
     )
   )
@@
     )
   )
+  (global_label "sda" (shape input) (at 53.34 96.52 180) (fields_autoplaced)
+    (effects (font (size 1.27 1.27)) (justify right))
+    (property "Intersheetrefs" "${INTERSHEET_REFS}" (at 47.0287 96.52 0)
+      (effects (font (size 1.27 1.27)) (justify right) hide)
+    )
+  )
   (global_label "c8" (shape input) (at 71.12 54.61 0) (fields_autoplaced)
     (effects (font (size 1.27 1.27)) (justify left))
@@
     )
   )
+  (global_label "scl" (shape input) (at 55.88 80.01 270) (fields_autoplaced)
+    (effects (font (size 1.27 1.27)) (justify right))
+    (property "Intersheetrefs" "${INTERSHEET_REFS}" (at 55.88 85.7771 90)
+      (effects (font (size 1.27 1.27)) (justify right) hide)
+    )
+  )
   (global_label "r1" (shape input) (at 93.98 86.36 180) (fields_autoplaced)
     (effects (font (size 1.27 1.27)) (justify right))
@@
     )
   )
+  (symbol (lib_id "power:+3.3V") (at 53.34 101.6 90) (unit 1)
+    (in_bom yes) (on_board yes) (dnp no) (fields_autoplaced)
+    (property "Reference" "#PWR03" (at 57.15 101.6 0)
+      (effects (font (size 1.27 1.27)) hide)
+    )
+    (property "Value" "+3.3V" (at 49.53 101.6 90)
+      (effects (font (size 1.27 1.27)) (justify left))
+    )
+    (property "Footprint" "" (at 53.34 101.6 0)
+      (effects (font (size 1.27 1.27)) hide)
+    )
+    (property "Datasheet" "" (at 53.34 101.6 0)
+      (effects (font (size 1.27 1.27)) hide)
+    )
+    (pin "1")
+    (instances
+      (project "qaz"
+        (path "/d7db0739-d565-4773-8b17-1b283fc7c7a9"
+          (reference "#PWR03") (unit 1)
+        )
+      )
+    )
+  )
   (symbol (lib_id "Switch:SW_Push") (at 165.1 100.33 0) (unit 1)
     (in_bom yes) (on_board yes) (dnp no) (fields_autoplaced)
@@
         (path "/d7db0739-d565-4773-8b17-1b283fc7c7a9"
           (reference "D13") (unit 1)
+        )
+      )
+    )
+  )
+  (symbol (lib_id "power:GND") (at 53.34 104.14 270) (unit 1)
+    (in_bom yes) (on_board yes) (dnp no) (fields_autoplaced)
+    (property "Reference" "#PWR02" (at 46.99 104.14 0)
+      (effects (font (size 1.27 1.27)) hide)
+    )
+    (property "Value" "GND" (at 49.53 104.14 90)
+      (effects (font (size 1.27 1.27)) (justify right))
+    )
+    (property "Footprint" "" (at 53.34 104.14 0)
+      (effects (font (size 1.27 1.27)) hide)
+    )
+    (property "Datasheet" "" (at 53.34 104.14 0)
+      (effects (font (size 1.27 1.27)) hide)
+    )
+    (pin "1")
+    (instances
+      (project "qaz"
+        (path "/d7db0739-d565-4773-8b17-1b283fc7c7a9"
+          (reference "#PWR02") (unit 1)
         )
       )
@@
         )
       )
+    )
+  )
+  (symbol (lib_id "display:OLED-128x32") (at 55.88 100.33 0) (unit 1)
+    (in_bom yes) (on_board yes) (dnp no) (fields_autoplaced)
+    (property "Reference" "J1" (at 72.39 99.06 0)
+      (effects (font (size 1.27 1.27)) (justify left))
+    )
+    (property "Value" "OLED-128x32" (at 72.39 101.6 0)
+      (effects (font (size 1.27 1.27)) (justify left))
+    )
+    (property "Footprint" "custom:OLED-128x32" (at 55.88 91.44 0)
+      (effects (font (size 1.27 1.27)) hide)
+    )
+    (property "Datasheet" "" (at 55.88 99.06 0)
+      (effects (font (size 1.27 1.27)) hide)
+    )
+    (pin "1")
+    (pin "2")
+    (pin "3")
+    (pin "4")
+    (instances
+      (project "qaz"
+        (path "/d7db0739-d565-4773-8b17-1b283fc7c7a9"
+          (reference "J1") (unit 1)
+        )
+      )
+    )
+  )
+  (symbol (lib_id "power:+3.3V") (at 45.72 59.69 90) (unit 1)
+    (in_bom yes) (on_board yes) (dnp no) (fields_autoplaced)
+    (property "Reference" "#PWR04" (at 49.53 59.69 0)
+      (effects (font (size 1.27 1.27)) hide)
+    )
+    (property "Value" "+3.3V" (at 41.91 59.69 90)
+      (effects (font (size 1.27 1.27)) (justify left))
+    )
+    (property "Footprint" "" (at 45.72 59.69 0)
+      (effects (font (size 1.27 1.27)) hide)
+    )
+    (property "Datasheet" "" (at 45.72 59.69 0)
+      (effects (font (size 1.27 1.27)) hide)
+    )
+    (pin "1")
+    (instances
+      (project "qaz"
+        (path "/d7db0739-d565-4773-8b17-1b283fc7c7a9"
+          (reference "#PWR04") (unit 1)
+        )
+      )
