File: art/art.kicad_pcb (KiCad board)
At the start: 2 copper layers, 92.6 x 34.2 mm, 14 parts, among them J1 AudioJack4, SW1 SW_Push, SW2 SW_Push, SW3 SW_Push, SW4 SW_Push, SW5 SW_Push, SW6 SW_Push, SW7 SW_Push, SW8 SW_Push, U1 rp2040-zero

Commit message: .
Connections:
- D1 pad 3: Net-(D1-K) -> r1
- D2 pad 3: Net-(D1-K) -> r1
- D3 pad 3: Net-(D3-K) -> r2
- D4 pad 3: Net-(D3-K) -> r2
- J1 pad R1: unconnected-(J1-PadR1) -> Net-(U1-13)
- J1 pad R2: unconnected-(J1-PadR2) -> Net-(U1-12)
- J1 pad S: unconnected-(J1-PadS) -> GND
- J1 pad T: unconnected-(J1-PadT) -> +3V3
- SW1 pad 2: Net-(SW1-Pad2) -> c1
- SW2 pad 2: Net-(SW2-Pad2) -> c2
- SW3 pad 2: Net-(SW3-Pad2) -> c3
- SW4 pad 2: Net-(SW4-Pad2) -> c4
- SW5 pad 2: Net-(SW1-Pad2) -> c1
- SW6 pad 2: Net-(SW2-Pad2) -> c2
- SW7 pad 2: Net-(SW3-Pad2) -> c3
- SW8 pad 2: Net-(SW4-Pad2) -> c4
- U1 pad 13: unconnected-(U1-12-Pad13) -> Net-(U1-12)
- U1 pad 14: unconnected-(U1-13-Pad14) -> Net-(U1-13)
- U1 pad 15: unconnected-(U1-14-Pad15) -> r2
- U1 pad 16: unconnected-(U1-15-Pad16) -> c1
- U1 pad 17: unconnected-(U1-26-Pad17) -> c2
- U1 pad 18: unconnected-(U1-27-Pad18) -> c3
- U1 pad 19: unconnected-(U1-28-Pad19) -> c4
- U1 pad 20: unconnected-(U1-29-Pad20) -> r1
- U1 pad 21: unconnected-(U1-3V3-Pad21) -> +3V3
- U1 pad 22: unconnected-(U1-GND-Pad22) -> GND
Routing:
- net c1: track 0.00 -> 86.2 mm, vias 0 -> 1
- net c2: track 0.00 -> 69.0 mm, vias 0 -> 1
- net r2: track 0.00 -> 63.6 mm
- net r1: track 0.00 -> 60.4 mm
- net c3: track 0.00 -> 51.7 mm, vias 0 -> 1
- net Net-(D1-K): track 37.2 -> 0.00 mm
- net Net-(D3-K): track 37.1 -> 0.00 mm
- net c4: track 0.00 -> 34.6 mm, vias 0 -> 1
- net +3V3: track 0.00 -> 24.2 mm
- net Net-(U1-12): track 0.00 -> 11.0 mm
- net Net-(U1-13): track 0.00 -> 10.4 mm
- net Net-(D3-A-Pad2): track 10.0 -> 13.2 mm
- added copper zone on B.Cu, net GND
- added copper zone on F.Cu, net GND
- removed copper zone on B.Cu, net (none)
- removed copper zone on F.Cu, net (none)
