File: art/art.kicad_pcb (KiCad board)
At the start: 2 copper layers, 92.6 x 34.2 mm, 14 parts, among them J1 AudioJack4, SW1 SW_Push, SW2 SW_Push, SW3 SW_Push, SW4 SW_Push, SW5 SW_Push, SW6 SW_Push, SW7 SW_Push, SW8 SW_Push, U1 rp2040-zero

Commit message: .
Parts:
- added REF**: Mounting_Wuerth_WA-SMSI-M1.6_H2mm_9774020633, Mounting_Wuerth:Mounting_Wuerth_WA-SMSI-M1.6_H2mm_9774020633, F.Cu at (113.9, 61.7)
- added REF**: Mounting_Wuerth_WA-SMSI-M1.6_H2mm_9774020633, Mounting_Wuerth:Mounting_Wuerth_WA-SMSI-M1.6_H2mm_9774020633, F.Cu at (77.7, 61.8)
- added REF**: Mounting_Wuerth_WA-SMSI-M1.6_H2mm_9774020633, Mounting_Wuerth:Mounting_Wuerth_WA-SMSI-M1.6_H2mm_9774020633, F.Cu at (132.6, 75.5)
- moved D3 35.3 mm to (77.7, 75.4)
- moved D4 35.3 mm to (113.8, 75.4)
- moved SW1 35.3 mm to (68.6, 53.2)
- moved SW2 35.3 mm to (86.7, 53.2)
- moved SW3 35.3 mm to (104.8, 53.2)
- moved SW4 35.3 mm to (122.8, 53.2)
- moved SW5 35.3 mm to (68.6, 70.2)
- moved U1 35.3 mm to (142.0, 56.4)
- moved J1 35.3 mm to (142.3, 73.6)
- moved SW6 35.3 mm to (86.7, 70.2)
- moved SW7 35.3 mm to (104.8, 70.2)
- moved SW8 35.3 mm to (122.8, 70.2)
- moved D1 34.9 mm to (77.7, 57.3)
- moved D2 34.8 mm to (113.8, 57.1)
Routing:
- net r1: track 60.4 -> 61.4 mm
- net c3: track 51.7 -> 52.4 mm
- net c4: track 34.6 -> 35.3 mm
- net c2: track 69.0 -> 69.6 mm
- net c1: track 86.2 -> 86.8 mm
Other:
- board text added: "ART"
- board text added: "BY FELIX"
- board text added: "PAD"
