File: jnew/jigsaw.kicad_pcb (KiCad board)
At the start: 2 copper layers, 31 x 48.8 mm, 3 parts, among them SW1 SW_Push, SW2 SW_Push

Commit message: .
Parts:
- added D1: D, Diode_SMD:D_SOD-123, B.Cu at (146.9, 39.3)
- added D1: D, Diode_SMD:D_SOD-123, B.Cu at (120.5, 49.5)
- added D2: D, Diode_SMD:D_SOD-123, B.Cu at (149.2, 66.9)
- added D2: D, Diode_SMD:D_SOD-123, B.Cu at (213.1, 80.6)
- added REF**: mousebites 2mm, PCM_marbastlib-various:mousebites_2mm, F.Cu at (137.8, 41.9)
- added REF**: STAB_MX_2u, PCM_marbastlib-mx:STAB_MX_2u, F.Cu at (222.5, 79.4)
- added REF**: mousebites 2mm, PCM_marbastlib-various:mousebites_2mm, F.Cu at (154.6, 58.7)
- added REF**: STAB_MX_2u, PCM_marbastlib-mx:STAB_MX_2u, F.Cu at (139.8, 68.1)
- added SW1: SW_Push, PCM_Switch_Keyboard_Hotswap_Kailh:SW_Hotswap_Kailh_MX_1.00u, F.Cu at (149.3, 47.1)
- added SW1: SW_Push, PCM_Switch_Keyboard_Hotswap_Kailh:SW_Hotswap_Kailh_MX_1.00u, F.Cu at (128.3, 47.1)
- added SW2: SW_Push, PCM_Switch_Keyboard_Hotswap_Kailh:SW_Hotswap_Kailh_MX_2.00u, F.Cu at (139.8, 68.1)
- moved SW1 173.5 mm to (222.7, 43.6)
- moved D1 173.5 mm to (214.9, 45.9)
- moved SW2 173.4 mm to (222.5, 79.4)
Routing:
- net row: track 23.6 -> 139.5 mm, vias 4 -> 6
- net col: track 65.9 -> 157.4 mm
- net Net-(D2-A): track 1.48 -> 10.8 mm
- net Net-(D1-A): track 3.51 -> 10.5 mm
Other:
- board size 31 x 48.8 mm -> 125.7 x 57.8 mm
