File: jnew/jigsaw.kicad_sch (KiCad schematic)
At the start: 6 parts, among them SW1 SW_Push

Commit message: .
Parts:
- removed TP1, TP2: TestPoint, TestPoint:TestPoint_Pad_D2.5mm, symbol Connector:TestPoint
- removed TP3, TP4: TestPoint, TestPoint:TestPoint_Pad_D4.0mm, symbol Connector:TestPoint
- added D2: D, Diode_SMD:D_SOD-123, symbol Device:D
- added SW2: SW_Push, PCM_Switch_Keyboard_Hotswap_Kailh:SW_Hotswap_Kailh_MX_2.00u, symbol Switch:SW_Push
- D1: footprint Diode_SMD:D_0603_1608Metric -> Diode_SMD:D_SOD-123
Connections:
- net row: now reaches D1.1 (K)
- net row: now also D2.1 (K)
- net col: now reaches SW1.2
- net col: now also SW2.2
- new net: D2.2 (A), SW2.1
Changed lines of the file:
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@@
 (kicad_sch (version 20230121) (generator eeschema)
   (paper "A4")
-  (junction (at 44.45 45.72) (diameter 0) (color 0 0 0 0)
+  (global_label "row" (shape input) (at 44.45 45.72 270) (fields_autoplaced)
+    (effects (font (size 1.27 1.27)) (justify right))
+    (property "Intersheetrefs" "${INTERSHEET_REFS}" (at 44.45 51.9709 90)
+      (effects (font (size 1.27 1.27)) (justify right) hide)
+    )
   )
-  (junction (at 54.61 38.1) (diameter 0) (color 0 0 0 0)
+  (global_label "col" (shape input) (at 54.61 38.1 270) (fields_autoplaced)
+    (effects (font (size 1.27 1.27)) (justify right))
+    (property "Intersheetrefs" "${INTERSHEET_REFS}" (at 54.61 43.988 90)
+      (effects (font (size 1.27 1.27)) (justify right) hide)
+    )
+  )
+  (global_label "col" (shape input) (at 72.39 39.37 270) (fields_autoplaced)
+    (effects (font (size 1.27 1.27)) (justify right))
+    (property "Intersheetrefs" "${INTERSHEET_REFS}" (at 72.39 45.258 90)
+      (effects (font (size 1.27 1.27)) (justify right) hide)
+    )
+  )
+  (global_label "row" (shape input) (at 62.23 46.99 270) (fields_autoplaced)
+    (effects (font (size 1.27 1.27)) (justify right))
+    (property "Intersheetrefs" "${INTERSHEET_REFS}" (at 62.23 53.2409 90)
+      (effects (font (size 1.27 1.27)) (justify right) hide)
+    )
   )
   (symbol (lib_id "Device:D") (at 44.45 41.91 90) (unit 1)
@@
       (effects (font (size 1.27 1.27)) (justify right))
     )
-    (property "Footprint" "Diode_SMD:D_0603_1608Metric" (at 44.45 41.91 0)
+    (property "Footprint" "Diode_SMD:D_SOD-123" (at 44.45 41.91 0)
       (effects (font (size 1.27 1.27)) hide)
     )
@@
     )
   )
-  (symbol (lib_id "Connector:TestPoint") (at 44.45 45.72 270) (unit 1)
+  (symbol (lib_id "Device:D") (at 62.23 43.18 90) (unit 1)
     (in_bom yes) (on_board yes) (dnp no) (fields_autoplaced)
-    (property "Reference" "TP2" (at 49.53 44.45 90)
-      (effects (font (size 1.27 1.27)) (justify left))
+    (property "Reference" "D2" (at 64.77 41.91 90)
+      (effects (font (size 1.27 1.27)) (justify right))
     )
-    (property "Value" "TestPoint" (at 49.53 46.99 90)
-      (effects (font (size 1.27 1.27)) (justify left))
+    (property "Value" "D" (at 64.77 44.45 90)
+      (effects (font (size 1.27 1.27)) (justify right))
     )
-    (property "Footprint" "TestPoint:TestPoint_Pad_D2.5mm" (at 44.45 50.8 0)
+    (property "Footprint" "Diode_SMD:D_SOD-123" (at 62.23 43.18 0)
       (effects (font (size 1.27 1.27)) hide)
     )
-    (property "Datasheet" "~" (at 44.45 50.8 0)
+    (property "Datasheet" "~" (at 62.23 43.18 0)
+      (effects (font (size 1.27 1.27)) hide)
+    )
+    (property "Sim.Device" "D" (at 62.23 43.18 0)
+      (effects (font (size 1.27 1.27)) hide)
+    )
+    (property "Sim.Pins" "1=K 2=A" (at 62.23 43.18 0)
       (effects (font (size 1.27 1.27)) hide)
     )
     (pin "1")
+    (pin "2")
     (instances
       (project "jigsaw"
         (path "/2389c087-2486-4304-a2e1-2b47c84a66a2"
-          (reference "TP2") (unit 1)
+          (reference "D2") (unit 1)
         )
       )
     )
   )
-  (symbol (lib_id "Connector:TestPoint") (at 54.61 38.1 270) (unit 1)
+  (symbol (lib_id "Switch:SW_Push") (at 67.31 39.37 0) (unit 1)
     (in_bom yes) (on_board yes) (dnp no) (fields_autoplaced)
-    (property "Reference" "TP3" (at 59.69 36.83 90)
-      (effects (font (size 1.27 1.27)) (justify left))
+    (property "Reference" "SW2" (at 67.31 31.75 0)
+      (effects (font (size 1.27 1.27)))
     )
-    (property "Value" "TestPoint" (at 59.69 39.37 90)
-      (effects (font (size 1.27 1.27)) (justify left))
+    (property "Value" "SW_Push" (at 67.31 34.29 0)
+      (effects (font (size 1.27 1.27)))
     )
-    (property "Footprint" "TestPoint:TestPoint_Pad_D4.0mm" (at 54.61 43.18 0)
+    (property "Footprint" "PCM_Switch_Keyboard_Hotswap_Kailh:SW_Hotswap_Kailh_MX_2.00u" (at 67.31 34.29 0)
       (effects (font (size 1.27 1.27)) hide)
     )
-    (property "Datasheet" "~" (at 54.61 43.18 0)
+    (property "Datasheet" "~" (at 67.31 34.29 0)
       (effects (font (size 1.27 1.27)) hide)
     )
     (pin "1")
+    (pin "2")
     (instances
       (project "jigsaw"
         (path "/2389c087-2486-4304-a2e1-2b47c84a66a2"
-          (reference "TP3") (unit 1)
+          (reference "SW2") (unit 1)
         )
       )
-    )
-  )
-  (symbol (lib_id "Connector:TestPoint") (at 44.45 45.72 180) (unit 1)
-    (in_bom yes) (on_board yes) (dnp no) (fields_autoplaced)
-    (property "Reference" "TP4" (at 46.99 47.752 0)
-      (effects (font (size 1.27 1.27)) (justify right))
-    )
-    (property "Value" "TestPoint" (at 46.99 50.292 0)
-      (effects (font (size 1.27 1.27)) (justify right))
-    )
-    (property "Footprint" "TestPoint:TestPoint_Pad_D4.0mm" (at 39.37 45.72 0)
-      (effects (font (size 1.27 1.27)) hide)
-    )
-    (property "Datasheet" "~" (at 39.37 45.72 0)
-      (effects (font (size 1.27 1.27)) hide)
-    )
-    (pin "1")
-    (instances
-      (project "jigsaw"
-        (path "/2389c087-2486-4304-a2e1-2b47c84a66a2"
-          (reference "TP4") (unit 1)
-        )
-      )
-    )
-  )
-  (symbol (lib_id "Connector:TestPoint") (at 54.61 38.1 0) (unit 1)
-    (in_bom yes) (on_board yes) (dnp no) (fields_autoplaced)
-    (property "Reference" "TP1" (at 57.15 33.528 0)
-      (effects (font (size 1.27 1.27)) (justify left) hide)
-    )
-    (property "Value" "TestPoint" (at 57.15 36.068 0)
-      (effects (font (size 1.27 1.27)) (justify left) hide)
-    )
-    (property "Footprint" "TestPoint:TestPoint_Pad_D2.5mm" (at 59.69 38.1 0)
-      (effects (font (size 1.27 1.27)) hide)
-    )
-    (property "Datasheet" "~" (at 59.69 38.1 0)
-      (effects (font (size 1.27 1.27)) hide)
-    )
-    (pin "1")
-    (instances
-      (project "jigsaw"
-        (path "/2389c087-2486-4304-a2e1-2b47c84a66a2"
-          (reference "TP1") (unit 1)
-        )
-      )

Commit message: .
Parts:
- added C1, C2: 22pf, Capacitor_SMD:C_0805_2012Metric, symbol Device:C
- added C3: 1uf, Capacitor_SMD:C_0805_2012Metric, symbol Device:C
- added D3, D4: D, Diode_SMD:D_SOD-123, symbol Device:D
- added R1, R4: 10k, Resistor_SMD:R_0805_2012Metric, symbol Device:R
- added R2, R3: 22, Resistor_SMD:R_0805_2012Metric, symbol Device:R
- added SW3, SW4: SW_Push, PCM_Switch_Keyboard_Hotswap_Kailh:SW_Hotswap_Kailh_MX_1.00u, symbol Switch:SW_Push
- added SW5: reset, symbol Switch:SW_Push
- added U1: ATmega32U2-A, Package_QFP:TQFP-32_7x7mm_P0.8mm, symbol MCU_Microchip_ATmega:ATmega32U2-A
- added Y1: 16MHz, Crystal:Crystal_SMD_3225-4Pin_3.2x2.5mm, symbol Device:Crystal_GND24_Small
Connections:
- net col: now also SW3.2, SW4.2
- net row: now also D3.1 (K), D4.1 (K)
- new net: C2.2, U1.1 (XTAL1), Y1.1
- new net: R4.1, U1.13 (~{HWB}/PD7)
- new net: R2.2, U1.29 (D+)
- new net: R1.2, SW5.2, U1.24 (PC1/~{RESET})
- new net: C1.2, U1.2 (PC0/XTAL2), Y1.3
- new net: C3.2, U1.27 (UCAP)
- new net: R3.2, U1.30 (D-)
- new net: D4.2 (A), SW4.1
- new net: D3.2 (A), SW3.1
- new net +5V: R1.1, U1.31 (UVCC), U1.32 (AVCC), U1.4 (VCC)
- new net GND: C1.1, C2.1, C3.1, R4.2, SW5.1, U1.28 (UGND), U1.3 (GND), Y1.2, Y1.4
- new net d+: R2.1
- new net d-: R3.1
