File: fuckit/fuckit.kicad_pcb (KiCad board)
At the start: 2 copper layers, 228.7 x 57.2 mm, 172 parts, among them SW1 SW_Push_45deg, SW10 SW_Push_45deg, SW100 SW_Push_45deg, SW101 SW_Push_45deg, SW102 SW_Push_45deg, SW103 SW_Push_45deg, SW104 SW_Push_45deg, SW105 SW_Push_45deg, SW106 SW_Push_45deg, SW107 SW_Push_45deg, SW108 SW_Push_45deg, SW109 SW_Push_45deg, SW11 SW_Push_45deg, SW110 SW_Push_45deg, SW111 SW_Push_45deg, SW112 SW_Push_45deg, SW113 SW_Push_45deg, SW114 SW_Push_45deg, SW115 SW_Push_45deg, SW116 SW_Push_45deg, SW117 SW_Push_45deg, SW118 SW_Push_45deg, SW119 SW_Push_45deg, SW12 SW_Push_45deg, SW120 SW_Push_45deg, SW121 SW_Push_45deg, SW122 SW_Push_45deg, SW123 SW_Push_45deg, SW124 SW_Push_45deg, SW125 SW_Push_45deg, SW126 SW_Push_45deg, SW127 SW_Push_45deg, SW128 SW_Push_45deg, SW129 SW_Push_45deg, SW13 SW_Push_45deg, SW130 SW_Push_45deg, SW131 SW_Push_45deg, SW132 SW_Push_45deg, SW133 SW_Push_45deg, SW134 SW_Push_45deg, SW135 SW_Push_45deg, SW14 SW_Push_45deg, SW15 SW_Push_45deg, SW16 SW_Push_45deg, SW17 SW_Push_45deg, SW18 SW_Push_45deg, SW19 SW_Push_45deg, SW2 SW_Push_45deg, SW20 SW_Push_45deg, SW21 SW_Push_45deg, SW22 SW_Push_45deg, SW23 SW_Push_45deg, SW24 SW_Push_45deg, SW25 SW_Push_45deg, SW26 SW_Push_45deg, SW27 SW_Push_45deg, SW28 SW_Push_45deg, SW29 SW_Push_45deg, SW3 SW_Push_45deg, SW30 SW_Push_45deg, SW31 SW_Push_45deg, SW32 SW_Push_45deg, SW33 SW_Push_45deg, SW34 SW_Push_45deg, SW35 SW_Push_45deg, SW36 SW_Push_45deg, SW37 SW_Push_45deg, SW38 SW_Push_45deg, SW39 SW_Push_45deg, SW4 SW_Push_45deg, SW40 SW_Push_45deg, SW41 SW_Push_45deg, SW42 SW_Push_45deg, SW43 SW_Push_45deg, SW44 SW_Push_45deg, SW45 SW_Push_45deg, SW46 SW_Push_45deg, SW47 SW_Push_45deg, SW48 SW_Push_45deg, SW49 SW_Push_45deg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

Commit message: .
Other:
- board text added: "PCB3D_BR_KBD"
- board text added: "PCB3D_TL_KBD"
Changed lines of the file:
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@@
       (outputformat 1)
       (mirror false)
-      (drillshape 1)
+      (drillshape 0)
       (scaleselection 1)
-      (outputdirectory "")
+      (outputdirectory "gerber/")
     )
   )
@@
   (gr_arc (start 245.345157 15.676602) (mid 247.466504 16.555267) (end 248.345157 18.676602)
     (stroke (width 0.1) (type default)) (layer "Edge.Cuts"))
+  (gr_text "PCB3D_BR_KBD" (at 248.444376 73.025184) (layer "User.9")
+    (effects (font (size 1.5 1.5) (thickness 0.3) bold) (justify right top))
+  )
+  (gr_text "PCB3D_TL_KBD" (at 19.546143 15.577383) (layer "User.9")
+    (effects (font (size 1.5 1.5) (thickness 0.3) bold) (justify left bottom))
+  )
   (segment (start 26.647335 22.721151) (end 39.687564 22.721151) (width 0.25) (layer "B.Cu") (net 1))
   (segment (start 22.82037 27.212929) (end 22.82037 24.46933) (width 0.25) (layer "B.Cu") (net 1))
