File: Alice30/Alice30.kicad_pcb (KiCad board)
At the start: 2 copper layers, 245.8 x 87.4 mm, 79 parts, among them J1 USB_B_Mini, SW1 SW_Push_45deg, SW10 SW_Push_45deg, SW11 SW_Push_45deg, SW12 SW_Push_45deg, SW13 SW_Push_45deg, SW14 SW_Push_45deg, SW15 SW_Push_45deg, SW16 SW_Push_45deg, SW17 SW_Push_45deg, SW18 SW_Push_45deg, SW19 SW_Push_45deg, SW2 SW_Push_45deg, SW20 SW_Push_45deg, SW21 SW_Push_45deg, SW22 SW_Push_45deg, SW23 SW_Push_45deg, SW24 SW_Push_45deg, SW25 SW_Push_45deg, SW26 SW_Push_45deg, SW27 SW_Push_45deg, SW28 SW_Push_45deg, SW29 SW_Push_45deg, SW3 SW_Push_45deg, SW30 SW_Push_45deg, SW31 SW_Push_45deg, SW32 SW_Push_45deg, SW33 SW_Push_45deg, SW34 SW_Push_45deg, SW35 SW_Push, SW4 SW_Push_45deg, SW5 SW_Push_45deg, SW6 SW_Push_45deg, SW7 SW_Push_45deg, SW8 SW_Push_45deg, SW9 SW_Push_45deg, U1 ATmega32U2-A, Y1 Crystal_GND24_Small

Commit message: .
Parts:
- removed C1, C2: 22pf, Capacitor_SMD:C_0805_2012Metric_Pad1.18x1.45mm_HandSolder
- removed C3: 1uf, Capacitor_SMD:C_0805_2012Metric_Pad1.18x1.45mm_HandSolder
- removed D1, D10, D11, D12, D13, D14, D15, D16, D17, D18, D19, D2, D20, D21, D22, D23, D24, D25, D26, D27, D28, D29, D3, D30, D31, D32, D33, D34, D4, D5, D6, D7, D8, D9: D, custom-parts:D_TH
- removed J1: USB_B_Mini, custom-parts:Molex-0548190589
- removed R1, R2, R3, R4: 10k, Resistor_SMD:R_0805_2012Metric_Pad1.20x1.40mm_HandSolder
- removed the SW35 at (153.5, 96.1)
- removed U1: ATmega32U2-A, Package_QFP:TQFP-32_7x7mm_P0.8mm
- removed Y1: Crystal_GND24_Small, Crystal:Crystal_SMD_3225-4Pin_3.2x2.5mm_HandSoldering
- added SW23: SW_Push_45deg, custom-parts:MX_1U_Plate, F.Cu at (244.8, 61.2)
- SW1, SW10, SW11, SW12, SW14, SW15, SW16, SW17, SW18, SW19, SW2, SW20, SW21, SW22, SW3, SW4, SW5, SW6, SW7, SW8, SW9: footprint custom-parts:MX_1U -> custom-parts:MX_1U_Plate
- SW13: footprint custom-parts:MX_1.25U -> custom-parts:MX_1U_Plate
- SW24: renamed from SW23; footprint custom-parts:MX_1.75U -> custom-parts:MX_1U_Plate
- SW25: renamed from SW24; footprint custom-parts:MX_1.25U -> custom-parts:MX_1U_Plate
- SW26: renamed from SW25; footprint custom-parts:MX_1U -> custom-parts:MX_1U_Plate
- SW27: renamed from SW26; footprint custom-parts:MX_1U -> custom-parts:MX_1U_Plate
- SW28: renamed from SW27; footprint custom-parts:MX_1U -> custom-parts:MX_1U_Plate
- SW29: renamed from SW28; footprint custom-parts:MX_1U -> custom-parts:MX_1U_Plate
- SW30: renamed from SW29; footprint custom-parts:MX_1U -> custom-parts:MX_1U_Plate
- SW31: renamed from SW30; footprint custom-parts:MX_1.5U -> custom-parts:MX_1U_Plate
- SW32: renamed from SW31; footprint custom-parts:MX_1U -> custom-parts:MX_1U_Plate
- SW33: renamed from SW32; footprint custom-parts:MX_1U -> custom-parts:MX_1U_Plate
- SW34: renamed from SW33; footprint custom-parts:MX_1U -> custom-parts:MX_1U_Plate
- SW35: renamed from SW34; footprint custom-parts:MX_1.25U -> custom-parts:MX_1U_Plate
- moved SW24 10.1 mm to (266.3, 61.2)
- moved SW20 7.00 mm to (185.2, 66.8)
- moved SW28 7.00 mm to (98.7, 84.6)
- moved SW33 7.00 mm to (212.2, 82.6)
- moved SW34 7.00 mm to (231.2, 80.9)
- moved SW7 7.00 mm to (160.0, 51.8)
- moved SW10 7.00 mm to (218.1, 43.8)
- moved SW11 7.00 mm to (238.4, 42.1)
- moved SW3 7.00 mm to (73.6, 44.1)
- moved SW5 7.00 mm to (112.9, 47.7)
- moved SW9 7.00 mm to (199.1, 45.5)
- moved SW29 7.00 mm to (118.9, 87.5)
- moved SW30 7.00 mm to (137.7, 90.8)
- moved SW31 7.00 mm to (168.4, 89.1)
- moved SW15 7.00 mm to (76.7, 63.5)
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Routing:
- net r3: track 363.7 -> 0.00 mm, vias 1 -> 0
- net r1: track 267.3 -> 0.00 mm, vias 2 -> 0
- net r2: track 266.5 -> 0.00 mm
- net c12: track 186.3 -> 0.00 mm, vias 2 -> 0
- net c1: track 167.3 -> 0.00 mm
- net c11: track 161.9 -> 0.00 mm, vias 2 -> 0
- net c10: track 156.6 -> 0.00 mm, vias 2 -> 0
- net c2: track 145.6 -> 0.00 mm
- net c9: track 136.4 -> 0.00 mm, vias 1 -> 0
- net c3: track 123.4 -> 0.00 mm
- net c8: track 112.7 -> 0.00 mm, vias 1 -> 0
- net c4: track 102.6 -> 0.00 mm
- net +5V: track 85.7 -> 0.00 mm, vias 7 -> 0
- net c7: track 77.5 -> 0.00 mm, vias 1 -> 0
- net c5: track 75.6 -> 0.00 mm
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- removed copper zone on B.Cu, net GND
- removed copper zone on F.Cu, net GND
Other:
- board size 245.8 x 87.4 mm -> 255.4 x 69 mm
